File: Hardware/GPS_Frontend/GPS_Frontend.kicad_pcb (KiCad board)
At the start: 4 copper layers, 44.2 x 25.4 mm, 34 parts, among them J1 Pmod B, J2 Passive ANT, J3 Active ANT, SW1 SW_DIP_x02, SW2 SW_DIP_x01, U1 MAX2769ETI_, U2 TPS7A2030PDBVR, U3 TPS7A2030PDBVR, Y1 19.2 Mhz

Commit message: Version submitted for manufacturing
Parts:
- added C17: 10n, Capacitor_SMD:C_0603_1608Metric, F.Cu at (157.0, 103.5)
- added C18: 1u, Capacitor_SMD:C_0603_1608Metric, F.Cu at (162.8, 106.2)
- added C19: 1u, Capacitor_SMD:C_0603_1608Metric, F.Cu at (161.0, 105.7)
- added C20: 1u, Capacitor_SMD:C_0603_1608Metric, F.Cu at (163.3, 113.3)
- added C21: 1u, Capacitor_SMD:C_0603_1608Metric, F.Cu at (161.5, 113.3)
- J1: value Pmod B -> Pmod
Connections:
- U1 pad 16: /CLKOUT -> Net-(U1-CLKOUT)
Routing:
- net /CLKOUT: track 24.6 -> 17.9 mm
- net Net-(U1-CLKOUT): track 0.00 -> 5.22 mm
- net GND: track 36.6 -> 41.6 mm
- net +3.3V: track 26.2 -> 29.8 mm
- net +3VD: track 11.8 -> 13.3 mm
- net +3VA: track 27.3 -> 28.0 mm
- net /SCK: track 23.4 -> 24.2 mm
- net /DIN: track 22.0 -> 22.7 mm
Other:
- board text added: "JLCJLCJLCJLC"
